Commit message: changed fdir1 to 0 0 0

File: mybot_description/urdf/macros.xacro (robot description, xacro)
@@ -38,9 +38,9 @@
        </link>
         <gazebo reference="${lr}_wheel">
-          <mu1 value="1.0"/>
-          <mu2 value="1.0"/>
+          <mu1 value="100.0"/>
+          <mu2 value="100.0"/>
           <kp  value="10000000.0" />
           <kd  value="1.0" />
-          <fdir1 value="1 0 0"/>
+          <fdir1 value="0 0 0"/>
           <material>Gazebo/Black</material>
         </gazebo>

File: mybot_description/urdf/mybot.xacro (robot description, xacro)
@@ -9,5 +9,5 @@
   <xacro:property name="casterMass" value="5"/>
   <xacro:property name="wheelWidth" value="0.05"/>
-  <xacro:property name="wheelRadius" value="0.1"/>
+  <xacro:property name="wheelRadius" value="0.11"/>
   <xacro:property name="wheelPos" value="0.2"/>
   <xacro:property name="wheelMass" value="5"/>
